File: 001.brd (EAGLE design)
At the start: 81 x 80 mm, 27 parts, among them CN01 PWR5V, CN02 JD-VCC, CN03 TO-RLY, CN04 I2C-LCD, CN05 INPUT-A, CN06 INPUT-B, CN07 BUTTON-A, CN08 BUTTON-B, CN09 BUTTON-STOP, CN10 DELAY-VR, M1 ARDUINO-NANO-3.0

Commit message: 1N4007に変更
Parts:
- D1, D10, D2, D3, D4, D5, D6, D7, D8, D9: value 1N4004 -> 1N4007
Changed lines of the file:
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@@
 <attribute name="VALUE" x="72.644" y="68.834" size="1.27" layer="27" ratio="10" rot="R90"/>
 </element>
-<element name="D1" library="diode" library_urn="urn:adsk.eagle:library:210" package="DO41-10" package3d_urn="urn:adsk.eagle:package:43336/1" value="1N4004" x="69.85" y="58.42" smashed="yes" rot="R90">
+<element name="D1" library="diode" library_urn="urn:adsk.eagle:library:210" package="DO41-10" package3d_urn="urn:adsk.eagle:package:43336/1" value="1N4007" x="69.85" y="58.42" smashed="yes" rot="R90">
 <attribute name="NAME" x="68.199" y="56.388" size="1.27" layer="25" ratio="10" rot="R90"/>
 <attribute name="POPULARITY" value="82" x="119.38" y="77.47" size="1.778" layer="27" rot="R90" display="off"/>
 <attribute name="VALUE" x="72.644" y="56.388" size="1.27" layer="27" ratio="10" rot="R90"/>
 </element>
-<element name="D2" library="diode" library_urn="urn:adsk.eagle:library:210" package="DO41-10" package3d_urn="urn:adsk.eagle:package:43336/1" value="1N4004" x="81.28" y="63.5" smashed="yes" rot="R180">
+<element name="D2" library="diode" library_urn="urn:adsk.eagle:library:210" package="DO41-10" package3d_urn="urn:adsk.eagle:package:43336/1" value="1N4007" x="81.28" y="63.5" smashed="yes" rot="R180">
 <attribute name="NAME" x="83.312" y="61.849" size="1.27" layer="25" ratio="10" rot="R180"/>
 <attribute name="POPULARITY" value="82" x="49.53" y="113.03" size="1.778" layer="27" rot="R180" display="off"/>
 <attribute name="VALUE" x="83.312" y="66.294" size="1.27" layer="27" ratio="10" rot="R180"/>
 </element>
-<element name="D3" library="diode" library_urn="urn:adsk.eagle:library:210" package="DO41-10" package3d_urn="urn:adsk.eagle:package:43336/1" value="1N4004" x="78.74" y="15.24" smashed="yes">
+<element name="D3" library="diode" library_urn="urn:adsk.eagle:library:210" package="DO41-10" package3d_urn="urn:adsk.eagle:package:43336/1" value="1N4007" x="78.74" y="15.24" smashed="yes">
 <attribute name="NAME" x="76.708" y="16.891" size="1.27" layer="25" ratio="10"/>
 <attribute name="POPULARITY" value="82" x="123.19" y="-34.29" size="1.778" layer="27" display="off"/>
 <attribute name="VALUE" x="76.708" y="12.446" size="1.27" layer="27" ratio="10"/>
 </element>
-<element name="D4" library="diode" library_urn="urn:adsk.eagle:library:210" package="DO41-10" package3d_urn="urn:adsk.eagle:package:43336/1" value="1N4004" x="78.74" y="22.86" smashed="yes">
+<element name="D4" library="diode" library_urn="urn:adsk.eagle:library:210" package="DO41-10" package3d_urn="urn:adsk.eagle:package:43336/1" value="1N4007" x="78.74" y="22.86" smashed="yes">
 <attribute name="NAME" x="76.708" y="24.511" size="1.27" layer="25" ratio="10"/>
 <attribute name="POPULARITY" value="82" x="97.79" y="-34.29" size="1.778" layer="27" display="off"/>
 <attribute name="VALUE" x="76.708" y="20.066" size="1.27" layer="27" ratio="10"/>
 </element>
-<element name="D5" library="diode" library_urn="urn:adsk.eagle:library:210" package="DO41-10" package3d_urn="urn:adsk.eagle:package:43336/1" value="1N4004" x="78.74" y="31.75" smashed="yes">
+<element name="D5" library="diode" library_urn="urn:adsk.eagle:library:210" package="DO41-10" package3d_urn="urn:adsk.eagle:package:43336/1" value="1N4007" x="78.74" y="31.75" smashed="yes">
 <attribute name="NAME" x="76.708" y="33.401" size="1.27" layer="25" ratio="10"/>
 <attribute name="POPULARITY" value="82" x="110.49" y="-25.4" size="1.778" layer="27" display="off"/>
@@
 <attribute name="VALUE" x="39.37" y="43.18" size="1.27" layer="21" rot="R90"/>
 </element>
-<element name="D6" library="diode" library_urn="urn:adsk.eagle:library:210" package="DO41-10" package3d_urn="urn:adsk.eagle:package:43336/1" value="1N4004" x="78.74" y="39.37" smashed="yes">
+<element name="D6" library="diode" library_urn="urn:adsk.eagle:library:210" package="DO41-10" package3d_urn="urn:adsk.eagle:package:43336/1" value="1N4007" x="78.74" y="39.37" smashed="yes">
 <attribute name="NAME" x="76.708" y="41.021" size="1.27" layer="25" ratio="10"/>
 <attribute name="POPULARITY" value="82" x="78.74" y="39.37" size="1.778" layer="27" display="off"/>
 <attribute name="VALUE" x="76.708" y="36.576" size="1.27" layer="27" ratio="10"/>
 </element>
-<element name="D7" library="diode" library_urn="urn:adsk.eagle:library:210" package="DO41-10" package3d_urn="urn:adsk.eagle:package:43336/1" value="1N4004" x="78.74" y="46.99" smashed="yes">
+<element name="D7" library="diode" library_urn="urn:adsk.eagle:library:210" package="DO41-10" package3d_urn="urn:adsk.eagle:package:43336/1" value="1N4007" x="78.74" y="46.99" smashed="yes">
 <attribute name="NAME" x="76.708" y="48.641" size="1.27" layer="25" ratio="10"/>
 <attribute name="POPULARITY" value="82" x="78.74" y="46.99" size="1.778" layer="27" display="off"/>
 <attribute name="VALUE" x="76.708" y="44.196" size="1.27" layer="27" ratio="10"/>
 </element>
-<element name="D8" library="diode" library_urn="urn:adsk.eagle:library:210" package="DO41-10" package3d_urn="urn:adsk.eagle:package:43336/1" value="1N4004" x="78.74" y="54.61" smashed="yes">
+<element name="D8" library="diode" library_urn="urn:adsk.eagle:library:210" package="DO41-10" package3d_urn="urn:adsk.eagle:package:43336/1" value="1N4007" x="78.74" y="54.61" smashed="yes">
 <attribute name="NAME" x="76.708" y="56.261" size="1.27" layer="25" ratio="10"/>
 <attribute name="POPULARITY" value="82" x="78.74" y="54.61" size="1.778" layer="27" display="off"/>
@@
 <attribute name="VALUE" x="41.1988" y="23.114" size="1.27" layer="27" ratio="10" rot="R90"/>
 </element>
-<element name="D9" library="diode" library_urn="urn:adsk.eagle:library:210" package="DO41-10" package3d_urn="urn:adsk.eagle:package:43336/1" value="1N4004" x="54.61" y="13.97" smashed="yes" rot="R180">
+<element name="D9" library="diode" library_urn="urn:adsk.eagle:library:210" package="DO41-10" package3d_urn="urn:adsk.eagle:package:43336/1" value="1N4007" x="54.61" y="13.97" smashed="yes" rot="R180">
 <attribute name="NAME" x="56.642" y="12.319" size="1.27" layer="25" ratio="10" rot="R180"/>
 <attribute name="POPULARITY" value="82" x="54.61" y="13.97" size="1.778" layer="27" rot="R180" display="off"/>
 <attribute name="VALUE" x="56.642" y="16.764" size="1.27" layer="27" ratio="10" rot="R180"/>
 </element>
-<element name="D10" library="diode" library_urn="urn:adsk.eagle:library:210" package="DO41-10" package3d_urn="urn:adsk.eagle:package:43336/1" value="1N4004" x="41.91" y="13.97" smashed="yes" rot="R180">
+<element name="D10" library="diode" library_urn="urn:adsk.eagle:library:210" package="DO41-10" package3d_urn="urn:adsk.eagle:package:43336/1" value="1N4007" x="41.91" y="13.97" smashed="yes" rot="R180">
 <attribute name="NAME" x="43.942" y="12.319" size="1.27" layer="25" ratio="10" rot="R180"/>
 <attribute name="POPULARITY" value="82" x="41.91" y="13.97" size="1.778" layer="27" rot="R180" display="off"/>

Commit message: ソースコードと一緒に管理
Parts:
- removed D4, D5, D6, D7, D8: 1N4007, diode:DO41-10
- added CN11: INPUT-B, holly:B02B-XH
- added CN12: BUTTON-C, holly:B02B-XH
- added R3: (no value), rcl:0207/7
- added U$2: (no value), Toshiba-TLP222AF:TOSHIBA_TLP222A_F_0
- moved D3 62.1 mm to (25.4, -16.5)
Connections:
- net +5V renamed N$10
- removed net N$10 (its old number): CN03.P$2, D8.A
- removed net N$15: D7.C, D8.C, M1.J1.8
- new net N$1: CN03.P$4, CN03.P$5, M1.J1.7
- new net N$12: CN11.P$2, D3.C
- net 5V: now also D3.A
- net GND: now also CN12.P$2, U$2.2, U$2.3
- net N$11: now also CN03.P$6, CN03.P$7; no longer D5.C, D6.C
- net N$14: now also CN03.P$8, CN03.P$9; no longer D3.C, D4.C
- net N$3: now also CN03.P$2, CN03.P$3, M1.J1.8; no longer CN03.P$9, D3.A
- net N$6: now also M1.J1.12, U$2.4; no longer CN03.P$8, D4.A
- net N$7: now also CN11.P$1, R3.1; no longer CN03.P$7, D5.A
- net N$8: now also R3.2, U$2.1; no longer CN03.P$6, D6.A
- net N$9: now also CN12.P$1, M1.J2.15; no longer CN03.P$3, D7.A
Routing:
- net N$3: track 21.6 -> 0.00 mm
- net N$15: track 17.8 -> 0.00 mm
- net N$6: track 16.5 -> 0.00 mm
- net N$10 (its old number): track 15.2 -> 0.00 mm
- net N$11: track 33.3 -> 20.3 mm
- net N$10: track 24.7 -> 12.0 mm
- net N$14: track 40.6 -> 30.0 mm
- net N$9: track 10.2 -> 0.00 mm
- net N$8: track 10.2 -> 0.00 mm
- net N$7: track 10.2 -> 0.00 mm

Commit message: CAM初版
Parts:
- removed D10, D9: 1N4007, diode:DO41-10
- removed U$4: (no value), Toshiba-TLP222AF:TOSHIBA_TLP222A_F_0
- added D4, D5: 1N4007, diode:DO41-10
- added U$3: (no value), Toshiba-TLP222AF:TOSHIBA_TLP222A_F_0
- C1: value (none) -> 10uF
- C2: value (none) -> 0.1uF
- CN07: value BUTTON-A -> INPUT-C
- CN08: value BUTTON-B -> BTN-A
- CN09: value BUTTON-STOP -> BTN-B
- CN10: value DELAY-VR -> BTN-C; device holly:B03B-XH -> holly:B02B-XH
- CN11: value INPUT-B -> BTN-STOP
- CN12: value BUTTON-C -> DELAY-VR; device holly:B02B-XH -> holly:B03B-XH
- R1, R2, R3: value (none) -> 4.7k
- U$1: value (none) -> U1
- moved CN11 80.0 mm to (41.9, 59.7), turned to 270 degrees
- moved D3 55.1 mm to (68.6, 17.8), turned to 90 degrees
- moved CN07 51.8 mm to (41.9, 8.89)
- moved U$2 48.6 mm to (57.1, 31.8), turned to 90 degrees
- moved CN12 45.0 mm to (33.0, 19.1), turned to 270 degrees
- moved R3 34.7 mm to (40.6, 19.1), turned to 90 degrees
- moved D2 32.1 mm to (71.1, 33.0), turned to 90 degrees
- moved CN09 23.0 mm to (41.9, 48.3), turned to 270 degrees
- moved CN10 22.9 mm to (33.0, 55.9)
- moved U$1 19.2 mm to (57.1, 47.0), turned to 90 degrees
- moved R1 18.9 mm to (63.5, 19.1)
- moved CN02 18.0 mm to (78.7, 48.3), turned to 90 degrees
- moved CN08 17.6 mm to (33.0, 44.5), turned to 270 degrees
- moved CN03 17.3 mm to (77.5, 36.8)
- moved CN01 14.9 mm to (78.7, 57.1), turned to 90 degrees
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Connections:
- net N$10 renamed 5V_M
- net N$2 renamed 5V_B
- net 5V: now also CN12.P$1, D4.A, D5.A; no longer CN10.P$1, D10.A, D9.A
- net GND: now also CN10.P$2, CN11.P$2, CN12.P$3, U$3.2, U$3.3; no longer CN07.P$2, CN10.P$3, CN12.P$2, U$4.2, U$4.3
- net N$12: now also CN07.P$2, D5.C; no longer CN11.P$2, D3.C
- net N$17: now also U$2.4; no longer U$4.4
- net N$20: now also U$2.1; no longer U$4.1
- net N$22: now also D4.C; no longer D10.C
- net N$24: now also D3.C; no longer D9.C
- net N$25: now also CN11.P$1; no longer CN09.P$1
- net N$26: now also CN09.P$1; no longer CN08.P$1
- net N$27: now also CN08.P$1; no longer CN07.P$1
- net N$29: now also CN12.P$2; no longer CN10.P$2
- net N$6: now also U$3.4; no longer U$2.4
- net N$7: now also CN07.P$1; no longer CN11.P$1
- net N$8: now also U$3.1; no longer U$2.1
- net N$9: now also CN10.P$1; no longer CN12.P$1
Routing:
- net 5V: track 184.8 -> 110.5 mm
- net N$8: track 0.00 -> 43.6 mm
- net 5V_M: track 12.0 -> 44.4 mm
- net N$19: track 13.0 -> 39.8 mm
- net N$1: track 0.00 -> 25.3 mm
- net N$18: track 5.08 -> 29.6 mm
- net N$9: track 0.00 -> 22.4 mm
- net N$3: track 0.00 -> 21.7 mm
- net N$17: track 30.5 -> 10.5 mm
- net 5V_B: track 5.08 -> 23.9 mm
- net N$23: track 22.4 -> 6.88 mm
- net N$6: track 0.00 -> 13.5 mm
- net N$21: track 20.3 -> 6.88 mm
- net N$20: track 14.8 -> 6.66 mm
- net N$7: track 0.00 -> 6.88 mm
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Other:
- board size 81 x 80 mm -> 55.5 x 66 mm
- board text added: "Model-400 K2005111 HOLLY&Co.,Ltd."

Commit message: ヴァリスタ追加
Parts:
- added U$4, U$5, U$6, U$7, U$8, U$9: TNR10V471K, holly:08-043X78_VARI
- moved CN05 13.5 mm to (74.9, 0.00)
- moved CN06 10.2 mm to (58.4, 0.00)
- moved CN07 9.25 mm to (44.5, 0.00)
Connections:
- net GND: now also U$5.2, U$7.2, U$9.1
- net N$12: now also U$8.2
- net N$21: now also U$6.2, U$7.1
- net N$22: now also U$6.1
- net N$23: now also U$4.2, U$5.1
- net N$24: now also U$4.1
- net N$7: now also U$8.1, U$9.2
Routing:
- net N$23: track 6.88 -> 22.2 mm
- net N$21: track 6.88 -> 19.9 mm
- net N$7: track 6.88 -> 19.7 mm
- net N$24: track 5.39 -> 17.6 mm
- net N$22: track 5.39 -> 15.0 mm
- net N$12: track 5.39 -> 13.2 mm
Other:
- board size 55.5 x 66 mm -> 55.5 x 78.7 mm
