File: 001.kicad_pcb (KiCad board)
At the start: 2 copper layers, 55.4 x 78.8 mm, 36 parts, among them CN1 PWR5V, CN10 BTN-C, CN11 BTN-STOP, CN12 DELAY-VR, CN2 JD-VCC, CN3 TO-RLY, CN4 I2C-LCD, CN5 INPUT-A, CN6 INPUT-B, CN7 INPUT-C, CN8 BTN-A, CN9 BTN-B, M1 ARDUINO-NANO-3.0

Commit message: foot printを見直し中
Parts:
- D1, D2, D3, D4, D5: footprint Diode_THT:D_DO-41_SOD81_P10.16mm_Horizontal -> Di:D_DO-41_SOD81_P10.16mm_Horizontal
- R1, R2, R3: footprint 001:0207_7 -> R:R_Axial_DIN0207_L6.3mm_D2.5mm_P10.16mm_Horizontal
- U$4, U$5, U$6, U$7, U$8, U$9: footprint 001:08-043X78_VARI -> varistor:RV_Disc_D12mm_W3.9mm_P7.5mm
- moved U$9 9.40 mm to (128.3, 141.0)
- moved R3 6.51 mm to (133.4, 122.9)
- moved R1 6.25 mm to (156.3, 122.7)
- moved U$8 4.23 mm to (130.8, 127.0)
- moved U$6 4.14 mm to (152.4, 128.4)
- moved U$4 3.51 mm to (166.9, 128.4)
- moved U$7 2.29 mm to (143.7, 133.5)
- moved U$5 2.21 mm to (158.9, 133.4)
- moved CN5 1.09 mm to (166.6, 135.5)
- moved C1 0.25 mm to (163.8, 73.2)
Connections:
- C1 pad 2: (no net) -> GND
- D1 pad 2: /5V_M -> (no net)
- D2 pad 2: /5V_M -> (no net)
Routing:
- net Net-(CN5-PadP$1): track 22.2 -> 19.3 mm
- net Net-(CN6-PadP$1): track 19.9 -> 18.7 mm
- net /5V_MPU: track 117.1 -> 118.0 mm
- net Net-(CN7-PadP$1): track 19.7 -> 20.3 mm
- removed copper zone on B.Cu, net GND
Other:
- outline, holes or cut-outs redrawn

Commit message: ガーバーデータも出来た
Parts:
- removed U$6: TNR10V471K, varistor:RV_Disc_D12mm_W3.9mm_P7.5mm
- added RV3: TNR10V471K, varistor:RV_Disc_D12mm_W3.9mm_P7.5mm, F.Cu at (152.4, 128.4)
- D1, D2, D3, D4, D5: footprint Di:D_DO-41_SOD81_P10.16mm_Horizontal -> Diode_THT:D_DO-41_SOD81_P10.16mm_Horizontal
- U1: renamed from U$1; value U1 -> TOSHIBA_TLP222A
- U2: renamed from U$2; value TOSHIBA_TLP222A_F_SIMPLE -> TOSHIBA_TLP222A
- U3: renamed from U$3; value TOSHIBA_TLP222A_F_SIMPLE -> TOSHIBA_TLP222A
- moved RV6 7.68 mm to (129.8, 133.5), turned to 270 degrees
- moved RV5 7.60 mm to (138.3, 128.4), turned to 180 degrees
- moved R2 6.25 mm to (144.8, 122.7)
- moved D4 0.77 mm to (149.9, 123.2)
- moved D3 0.51 mm to (161.3, 123.2)
- moved D5 0.51 mm to (138.4, 123.2)
- moved D2 0.08 mm to (165.2, 87.7)
- renumbered U$4 to RV1, U$5 to RV2, U$7 to RV4, U$8 to RV5, U$9 to RV6
Connections:
- D1 pad 1: (no net) -> /5V_MPU
- D1 pad 2: (no net) -> /5V_M
- D2 pad 1: (no net) -> /5V_JDV
- D2 pad 2: (no net) -> /5V_M
- D3 pad 1: (no net) -> Net-(CN5-PadP$2)
- D3 pad 2: (no net) -> /5V_MPU
- D4 pad 1: (no net) -> Net-(CN6-PadP$2)
- D4 pad 2: (no net) -> /5V_MPU
- D5 pad 1: (no net) -> Net-(CN7-PadP$2)
- D5 pad 2: (no net) -> /5V_MPU
- RV5 pad 1: Net-(CN7-PadP$1) -> Net-(CN7-PadP$2)
- RV5 pad 2: Net-(CN7-PadP$2) -> Net-(CN7-PadP$1)
- RV6 pad 1: GND -> Net-(CN7-PadP$1)
- RV6 pad 2: Net-(CN7-PadP$1) -> GND
Routing:
- net Net-(CN7-PadP$1): track 20.3 -> 17.7 mm
- net Net-(CN6-PadP$1): track 18.7 -> 16.2 mm
- added copper zone on B.Cu, net (none)
