File: 001.kicad_pcb (KiCad board)
At the start: 2 copper layers, 55.4 x 78.8 mm, 36 parts, among them CN1 PWR5V, CN10 BTN-C, CN11 BTN-STOP, CN12 DELAY-VR, CN2 JD-VCC, CN3 TO-RLY, CN4 I2C-LCD, CN5 INPUT-A, CN6 INPUT-B, CN7 INPUT-C, CN8 BTN-A, CN9 BTN-B, M1 ARDUINO-NANO-3.0, U1 TOSHIBA_TLP222A, U2 TOSHIBA_TLP222A, U3 TOSHIBA_TLP222A

Commit message: フレームを追加とケースの加工データ
Routing:
- added copper zone on B.Cu, net GND
- removed copper zone on B.Cu, net (none)
