File: 001.sch (KiCad schematic (older format))
At the start: 32 parts, among them CN1 PWR5V, CN10 BTN-C, CN11 BTN-STOP, CN12 DELAY-VR, CN2 JD-VCC, CN3 TO-RLY, CN4 I2C-LCD, CN5 INPUT-A, CN6 INPUT-B, CN7 INPUT-C, CN8 BTN-A, CN9 BTN-B, M1 ARDUINO-NANO-3.0

Commit message: foot printを見直し中
Parts:
- removed C1: 10uF, C:CP_Radial_D5.0mm_P2.00mm, symbol 001-eagle-import:CPOL-EUE2-5
- added C1: 10uF, C:CP_Radial_D5.0mm_P2.00mm, symbol Device:CP
- D1, D2, D3, D4, D5: footprint Diode_THT:D_DO-41_SOD81_P10.16mm_Horizontal -> Di:D_DO-41_SOD81_P10.16mm_Horizontal
- R1, R2, R3: footprint 001:0207_7 -> R:R_Axial_DIN0207_L6.3mm_D2.5mm_P10.16mm_Horizontal
- U$4, U$5, U$6, U$7, U$8, U$9: footprint 001:08-043X78_VARI -> varistor:RV_Disc_D12mm_W3.9mm_P7.5mm
Connections:
- net 5V_M: now also C1.1
- net GND: now also C1.2
- no-connect marks 11 -> 13
Other:
- moved on the sheet: D1
Changed lines of the file:
@@
 EELAYER 30 0
 EELAYER END
-$Descr User 11774 8268
+$Descr A4 11693 8268
 encoding utf-8
 Sheet 1 1
-Title ""
-Date ""
-Rev ""
-Comp ""
-Comment1 ""
+Title "K2005111"
+Date "2020-06-26"
+Rev "001"
+Comp "HOLLY&Co.,Ltd."
+Comment1 "Designer: Masafumi Horimoto"
 Comment2 ""
 Comment3 ""
@@
 GND
 Wire Wire Line
-	7600 1100 7200 1100
+	7550 1100 7200 1100
 Wire Wire Line
 	7200 1100 7200 2000
@@
 	5000 5400 5900 5400
 Wire Wire Line
-	7800 1100 8100 1100
+	7750 1100 8100 1100
 Wire Wire Line
 	8100 1100 8100 2300
@@
 L 001-eagle-import:1N4004 D1
 U 1 1 52A85BB0
-P 7700 1100
-F 0 "D1" H 7800 1119 59  0000 L BNN
-F 1 "1N4007" H 7800 1009 59  0000 L BNN
-F 2 "Diode_THT:D_DO-41_SOD81_P10.16mm_Horizontal" H 7700 1100 50  0001 C CNN
-F 3 "" H 7700 1100 50  0001 C CNN
-	1    7700 1100
+P 7650 1100
+F 0 "D1" H 7750 1119 59  0000 L BNN
+F 1 "1N4007" H 7750 1009 59  0000 L BNN
+F 2 "Di:D_DO-41_SOD81_P10.16mm_Horizontal" H 7650 1100 50  0001 C CNN
+F 3 "" H 7650 1100 50  0001 C CNN
+	1    7650 1100
 	-1   0    0    1
 $EndComp
@@
 F 0 "D2" H 8500 2319 59  0000 L BNN
 F 1 "1N4007" H 8500 2209 59  0000 L BNN
-F 2 "Diode_THT:D_DO-41_SOD81_P10.16mm_Horizontal" H 8400 2300 50  0001 C CNN
+F 2 "Di:D_DO-41_SOD81_P10.16mm_Horizontal" H 8400 2300 50  0001 C CNN
 F 3 "" H 8400 2300 50  0001 C CNN
 	1    8400 2300
@@
 $EndComp
 $Comp
-L 001-eagle-import:CPOL-EUE2-5 C1
-U 1 1 D1512118
-P 9000 1300
-F 0 "C1" H 9045 1319 59  0000 L BNN
-F 1 "10uF" H 9045 1119 59  0000 L BNN
-F 2 "C:CP_Radial_D5.0mm_P2.00mm" H 9000 1300 50  0001 C CNN
-F 3 "" H 9000 1300 50  0001 C CNN
-	1    9000 1300
-	1    0    0    -1
-$EndComp
-$Comp
 L 001-eagle-import:C-EU025-025X050 C2
 U 1 1 B94C3227
@@
 F 0 "R1" H 2250 3559 59  0000 L BNN
 F 1 "4.7k" H 2250 3370 59  0000 L BNN
-F 2 "001:0207_7" H 2400 3500 50  0001 C CNN
+F 2 "R:R_Axial_DIN0207_L6.3mm_D2.5mm_P10.16mm_Horizontal" H 2400 3500 50  0001 C CNN
 F 3 "" H 2400 3500 50  0001 C CNN
 	1    2400 3500
@@
 F 0 "R2" H 2050 4859 59  0000 L BNN
 F 1 "4.7k" H 2050 4670 59  0000 L BNN
-F 2 "001:0207_7" H 2200 4800 50  0001 C CNN
+F 2 "R:R_Axial_DIN0207_L6.3mm_D2.5mm_P10.16mm_Horizontal" H 2200 4800 50  0001 C CNN
 F 3 "" H 2200 4800 50  0001 C CNN
 	1    2200 4800
@@
 F 0 "D3" H 2500 3219 59  0000 L BNN
 F 1 "1N4007" H 2500 3109 59  0000 L BNN
-F 2 "Diode_THT:D_DO-41_SOD81_P10.16mm_Horizontal" H 2400 3200 50  0001 C CNN
+F 2 "Di:D_DO-41_SOD81_P10.16mm_Horizontal" H 2400 3200 50  0001 C CNN
 F 3 "" H 2400 3200 50  0001 C CNN
 	1    2400 3200
@@
 F 0 "D4" H 2300 4419 59  0000 L BNN
 F 1 "1N4007" H 2300 4309 59  0000 L BNN
-F 2 "Diode_THT:D_DO-41_SOD81_P10.16mm_Horizontal" H 2200 4400 50  0001 C CNN
+F 2 "Di:D_DO-41_SOD81_P10.16mm_Horizontal" H 2200 4400 50  0001 C CNN
 F 3 "" H 2200 4400 50  0001 C CNN
 	1    2200 4400
@@
 F 0 "R3" H 2050 5959 59  0000 L BNN
 F 1 "4.7k" H 2150 5770 59  0000 L BNN
-F 2 "001:0207_7" H 2200 5900 50  0001 C CNN
+F 2 "R:R_Axial_DIN0207_L6.3mm_D2.5mm_P10.16mm_Horizontal" H 2200 5900 50  0001 C CNN
 F 3 "" H 2200 5900 50  0001 C CNN
 	1    2200 5900
@@
 F 0 "D5" H 2300 5619 59  0000 L BNN
 F 1 "1N4007" H 2300 5509 59  0000 L BNN
-F 2 "Diode_THT:D_DO-41_SOD81_P10.16mm_Horizontal" H 2200 5600 50  0001 C CNN
+F 2 "Di:D_DO-41_SOD81_P10.16mm_Horizontal" H 2200 5600 50  0001 C CNN
 F 3 "" H 2200 5600 50  0001 C CNN
 	1    2200 5600
@@
 F 0 "U$4" V 2000 3450 59  0000 L BNN
 F 1 "TNR10V471K" V 1880 3470 59  0000 L BNN
-F 2 "001:08-043X78_VARI" H 1900 3400 50  0001 C CNN
+F 2 "varistor:RV_Disc_D12mm_W3.9mm_P7.5mm" H 1900 3400 50  0001 C CNN
 F 3 "" H 1900 3400 50  0001 C CNN
 	1    1900 3400
@@
 F 0 "U$5" V 1920 3870 59  0000 L BNN
 F 1 "TNR10V471K" V 1810 3880 59  0000 L BNN
-F 2 "001:08-043X78_VARI" H 1900 3800 50  0001 C CNN
+F 2 "varistor:RV_Disc_D12mm_W3.9mm_P7.5mm" H 1900 3800 50  0001 C CNN
 F 3 "" H 1900 3800 50  0001 C CNN
 	1    1900 3800
@@
 F 0 "U$6" V 1880 4670 59  0000 L BNN
 F 1 "TNR10V471K" V 1780 4640 59  0000 L BNN
-F 2 "001:08-043X78_VARI" H 1800 4600 50  0001 C CNN
+F 2 "varistor:RV_Disc_D12mm_W3.9mm_P7.5mm" H 1800 4600 50  0001 C CNN
 F 3 "" H 1800 4600 50  0001 C CNN
 	1    1800 4600
@@
 F 0 "U$7" H 2180 5120 59  0000 R TNN
 F 1 "TNR10V471K" H 2360 5210 59  0000 R TNN
-F 2 "001:08-043X78_VARI" H 2000 5000 50  0001 C CNN
+F 2 "varistor:RV_Disc_D12mm_W3.9mm_P7.5mm" H 2000 5000 50  0001 C CNN
 F 3 "" H 2000 5000 50  0001 C CNN
 	1    2000 5000
@@
 F 0 "U$8" V 1580 5580 59  0000 R TNN
 F 1 "TNR10V471K" V 1690 5660 59  0000 R TNN
-F 2 "001:08-043X78_VARI" H 1700 5700 50  0001 C CNN
+F 2 "varistor:RV_Disc_D12mm_W3.9mm_P7.5mm" H 1700 5700 50  0001 C CNN
 F 3 "" H 1700 5700 50  0001 C CNN
 	1    1700 5700
@@
 F 0 "U$9" H 2060 6050 59  0000 R TNN
 F 1 "TNR10V471K" H 2230 5970 59  0000 R TNN
-F 2 "001:08-043X78_VARI" H 2000 6100 50  0001 C CNN
+F 2 "varistor:RV_Disc_D12mm_W3.9mm_P7.5mm" H 2000 6100 50  0001 C CNN
 F 3 "" H 2000 6100 50  0001 C CNN
 	1    2000 6100
@@
 Text Label 6850 1100 0    50   ~ 0
 5V_MPU
+Text Label 7800 1100 0    50   ~ 0
+5V_M
+Text Label 8150 2300 0    50   ~ 0
+5V_M
+Text Label 7450 950  0    50   ~ 0
+5V_MPU
+NoConn ~ 6600 3000
+NoConn ~ 6600 1700
+$Comp
+L Device:CP C1
+U 1 1 5EFE5C07
+P 9000 1350
+F 0 "C1" H 9118 1396 50  0000 L CNN
+F 1 "10uF" H 9118 1305 50  0000 L CNN
+F 2 "C:CP_Radial_D5.0mm_P2.00mm" H 9038 1200 50  0001 C CNN
+F 3 "~" H 9000 1350 50  0001 C CNN
+	1    9000 1350
+	1    0    0    -1
+$EndComp
 $EndSCHEMATC

Commit message: ガーバーデータも出来た
Parts:
- removed D1, D2, D3, D4, D5: 1N4007, Di:D_DO-41_SOD81_P10.16mm_Horizontal, symbol 001-eagle-import:1N4004
- added D1, D2, D3, D4, D5: 1N4007, Diode_THT:D_DO-41_SOD81_P10.16mm_Horizontal, symbol Diode:1N4007
- R1, R2, R3: symbol 001-eagle-import:R-US_0207_7 -> Device:R_US
- RV1: renamed from U$4; symbol 001-eagle-import:TNR10V471K -> Device:Varistor_US
- RV2: renamed from U$5; symbol 001-eagle-import:TNR10V471K -> Device:Varistor_US
- RV3: renamed from U$6; symbol 001-eagle-import:TNR10V471K -> Device:Varistor_US
- RV4: renamed from U$7; symbol 001-eagle-import:TNR10V471K -> Device:Varistor_US
- RV5: renamed from U$8; symbol 001-eagle-import:TNR10V471K -> Device:Varistor_US
- RV6: renamed from U$9; symbol 001-eagle-import:TNR10V471K -> Device:Varistor_US
- U1: renamed from U$1; value U1 -> TOSHIBA_TLP222A
- U2: renamed from U$2; value TOSHIBA_TLP222A_F_SIMPLE -> TOSHIBA_TLP222A
- U3: renamed from U$3; value TOSHIBA_TLP222A_F_SIMPLE -> TOSHIBA_TLP222A
Connections:
- net 5V_JDV: now also D2.1 (K)
- net 5V_M: now also D1.2 (A), D2.2 (A)
- net 5V_MPU: now also D1.1 (K), D3.2 (A), D4.2 (A), D5.2 (A)
- net GND: now also RV6.2; no longer RV6.1
- net at CN5.P$2 (1), RV1.1: now also D3.1 (K)
- net at CN6.P$2 (1), RV3.1: now also D4.1 (K)
- net at CN7.P$1 (1), R3.1: now also RV5.2, RV6.1; no longer RV5.1, RV6.2
- net at CN7.P$2 (1): now also RV5.1, D5.1 (K); no longer RV5.2
